Commit message: update 21.3.19

File: install/share/robotiq_2f_85_gripper_visualization/urdf/robotiq_arg2f_85_model.xacro (robot description, xacro)
@@ -2,4 +2,5 @@
 <robot name="robotiq_arg2f_85_model" xmlns:xacro="http://ros.org/wiki/xacro">
   <xacro:include filename="$(find robotiq_2f_85_gripper_visualization)/urdf/robotiq_arg2f_85_model_macro.xacro" />
+  <xacro:include filename="$(find robotiq_2f_85_gripper_visualization)/urdf/robotiq_arg2f.xacro" />
   <xacro:robotiq_arg2f_85 prefix=""/>
 </robot>

File: src/brendan_ur5e/urdf/brendan_ur5e.urdf.xacro (robot description, xacro)
@@ -8,9 +8,13 @@
   <xacro:include filename="$(find brendan_ur5e)/urdf/ur5e.urdf.xacro" />
   <!-- robotiq_2f_85 gripper -->
-  <xacro:include filename="$(find robotiq)/robotiq_2f_85_gripper_visualization/robotiq_arg2f_85_model.xacro" />
+  <!--
+  <xacro:include filename="$(find brendan_ur5e)/urdf/robotiq_arg2f_85_model_macro.xacro" />
+  <xacro:include filename="$(find brendan_ur5e)/urdf/robotiq_arg2f.xacro" />
+  -->
+  <xacro:include filename="($find brendan_ur5e)/urdf/robotiq_arg2f_85_model.urdf.xacro" />
   <!-- arm -->
   <xacro:ur5e_robot prefix="" joint_limited="false"/>
   <!-- gripper -->
-  <xacro:robotiq_arg2f prefix=""/>
+  <xacro:robotiq_arg2f_85 prefix=""/>
   <!-- world -->
   <link name="world" />
@@ -21,3 +25,9 @@
     <origin xyz="0.0 0.0 0.0" rpy="0.0 0.0 0.0" />
   </joint>
+  <!-- robot to gripper joint -->
+  <joint name="gripper_joint" type="fixed">
+    <parent link="ee_link" />
+    <child link = "robotiq_arg2f_base_link" />
+    <origin xyz="0 0 0" rpy="0 0 0"/>
+  </joint>
 </robot>

File: src/brendan_ur5e/urdf/ur5e.urdf.xacro (robot description, xacro)
@@ -1,4 +1,5 @@
 <?xml version="1.0"?>
-<robot xmlns:xacro="http://ros.org/wiki/xacro">
+<robot xmlns:xacro="http://ros.org/wiki/xacro"
+	name="arm">
   <xacro:include filename="$(find ur_e_description)/urdf/ur.transmission.xacro" />
   <xacro:include filename="$(find ur_e_description)/urdf/ur.gazebo.xacro" />
