Commit message: euwha

File: src/brendan_ur5e/urdf/brendan_ur5e.urdf.xacro (robot description, xacro)
@@ -8,9 +8,7 @@
   <xacro:include filename="$(find brendan_ur5e)/urdf/ur5e.urdf.xacro" />
   <!-- robotiq_2f_85 gripper -->
-  <!--
   <xacro:include filename="$(find brendan_ur5e)/urdf/robotiq_arg2f_85_model_macro.xacro" />
   <xacro:include filename="$(find brendan_ur5e)/urdf/robotiq_arg2f.xacro" />
-  -->
-  <xacro:include filename="($find brendan_ur5e)/urdf/robotiq_arg2f_85_model.urdf.xacro" />
+  <!--<xacro:include filename="$(find brendan_ur5e)/urdf/robotiq_arg2f_85_model.urdf.xacro" />-->
   <!-- arm -->
   <xacro:ur5e_robot prefix="" joint_limited="false"/>
@@ -25,9 +23,9 @@
     <origin xyz="0.0 0.0 0.0" rpy="0.0 0.0 0.0" />
   </joint>
-  <!-- robot to gripper joint -->
+  <!-- robot to gripper joint
   <joint name="gripper_joint" type="fixed">
     <parent link="ee_link" />
     <child link = "robotiq_arg2f_base_link" />
     <origin xyz="0 0 0" rpy="0 0 0"/>
-  </joint>
+  </joint>-->
 </robot>

File: src/brendan_ur5e/urdf/robotiq_arg2f.xacro (robot description, xacro)
@@ -24,4 +24,10 @@
       </collision>
     </link>
+    <!-- robot to gripper joint -->
+    <joint name="gripper_joint" type="fixed">
+      <parent link="${prefix}ee_link" />
+      <child link = "${prefix}robotiq_arg2f_base_link" />
+      <origin xyz="0 0 0" rpy="0 ${pi / 2.0} 0"/>
+    </joint>
   </xacro:macro>
   <xacro:macro name="finger_joints" params="prefix fingerprefix reflect">

File: src/brendan_ur5e/urdf/ur5e_gripper_no_macros.urdf.xacro (robot description, xacro)
@@ -2,4 +2,6 @@
 <robot xmlns:xacro="http://ros.org/wiki/xacro"
        name="ur5e" >
+   <!-- world -->
+  <link name="world" />
   <xacro:property name="prefix" value=""/>
   <xacro:property name="joint_limited" value="false"/>
@@ -670,6 +672,4 @@
       <mimic joint="${prefix}finger_joint" multiplier="1" offset="0" />
     </joint>
-   <!-- world -->
-  <link name="world" />
   <!-- world to robot joint -->
   <joint name="world_joint" type="fixed">
